File: src/noise_monitor.brd (EAGLE design)
At the start: 53 x 48 mm, 70 parts, among them IC2 MCP73831/OT, T1 S8050, T2 S8050, U2 TEXAS_INSTRUMENTS_SN74HC125TE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, U4 ESP8266-12E/ESP-12E, U5 CP2102N-A02-GQFN28, U6 LP2989AILD-3.3, X2 SIMLOCK-C707_10M006_512_2

Commit message: Fixed DRC
Parts:
- removed MICRO_USB: 10118192-0001LF, noise_tracker:AMPHENOL_10118192-0001LF
- removed S1, S2: KMR621NGLFS, AQ_sensor_GSM:SW_KMR621NGLFS
- added D7: ON_SEMI_1N4148WSON_SEMI_1N4148WS_0_0, noise_monitor:ON_SEMI_1N4148WS_0
- added FLASH, RESET: KMR621NGLFS, noise_monitor:SW_KMR621NGLFS
- added MICRO-USB: 10118192-0001LF, noise_monitor:AMPHENOL_10118192-0001LF
- added R23: 0R, rcl:R0201
- CN1: device AQ_sensor_GSM:JST-PH-2-SMT-RA -> noise_monitor:JST-PH-2-SMT-RA
- D1, D4: device noise_tracker:ON_SEMI_1N4148WS_0 -> noise_monitor:ON_SEMI_1N4148WS_0
- D2: device noise_tracker:ON_SEMICONDUCTOR_MMSZ5231BT1G_0 -> noise_monitor:ON_SEMICONDUCTOR_MMSZ5231BT1G_0
- D3: device noise_tracker:SEMTECH_SMF05C_0 -> noise_monitor:SEMTECH_SMF05C_0
- D5, D6: device AQ_sensor_GSM:ON_SEMI_1N4148WS_0 -> noise_monitor:ON_SEMI_1N4148WS_0
- IC2: device noise_tracker:SOT23-5L -> noise_monitor:SOT23-5L
- MK2: device noise_tracker:MIC_SPH0645LM4H-B -> noise_monitor:MIC_SPH0645LM4H-B
- POWER: device AQ_sensor_GSM:SW_PCM12SMTR -> noise_monitor:SW_PCM12SMTR
- T1, T2: device noise_tracker:SC59-BEC -> noise_monitor:SC59-BEC
- U1: device noise_tracker:SIM800L -> noise_monitor:SIM800L
- U2: device noise_tracker:TEXAS_INSTRUMENTS_SN74HC125_0 -> noise_monitor:TEXAS_INSTRUMENTS_SN74HC125_0
- U4: device noise_tracker:XCVR_ESP8266-12E/ESP-12E -> noise_monitor:XCVR_ESP8266-12E/ESP-12E
- U5: device CP2102N-A02-GQFN28:QFN50P500X500X80-29N -> noise_monitor:QFN50P500X500X80-29N
- U6: device LP2989AILD-3.3:DFN400X400X80-9N -> noise_monitor:DFN400X400X80-9N
- X1: device AQ_sensor_GSM:SMA_EDGELAUNCH_UFL -> noise_monitor:SMA_EDGELAUNCH_UFL
- X2: device noise_tracker:C707_10M006_512_2 -> noise_monitor:C707_10M006_512_2
- moved D4 1.52 mm to (42.5, 39.1), turned to 90 degrees
- moved C3 1.27 mm to (45.2, 26.5), turned to 0 degrees
- moved C12 0.89 mm to (12.6, 18.0)
- moved C13 0.76 mm to (12.2, 20.1)
- moved R1 0.62 mm to (38.3, 31.0)
- moved R7 0.54 mm to (38.4, 38.7)
- moved R6 0.45 mm to (38.4, 35.4)
- moved FULL 0.25 mm to (6.99, 29.6)
- moved NET 0.10 mm to (38.6, 33.8)
- renumbered CRG to CHRG, TP1 to 5V, TP2 to GND, TP3 to 3V3, TP4 to V-LIPO
Connections:
- net V_BUS renamed VB
- removed net VBUS: MICRO_USB.1, POWER.1
- new net N$1: C12.2, C13.2, R23.2, U5.6
- new net V_IN: D7.1, MICRO-USB.1, POWER.1
- net +3V3: now also R23.1; no longer C12.2, C13.2, U5.6
- net D+: now also MICRO-USB.3; no longer MICRO_USB.3
- net D-: now also MICRO-USB.2; no longer MICRO_USB.2
- net ESP_RST: now also RESET.1_1, RESET.1_2; no longer S2.1_1, S2.1_2
- net GND: now also D7.2, FLASH.2_1, FLASH.2_2, MICRO-USB.4, MICRO-USB.5, MICRO-USB.SH1, MICRO-USB.SH2, MICRO-USB.SH3, MICRO-USB.SH4, MICRO-USB.SH5, MICRO-USB.SH6, RESET.2_1, RESET.2_2; no longer MICRO_USB.4, MICRO_USB.5, MICRO_USB.SH1, MICRO_USB.SH2, MICRO_USB.SH3, MICRO_USB.SH4, MICRO_USB.SH5, MICRO_USB.SH6, S1.2_1, S1.2_2, S2.2_1, S2.2_2
- net IO0: now also FLASH.1_1, FLASH.1_2; no longer S1.1_1, S1.1_2
Routing:
- net DTR: track 1.76 -> 33.1 mm, vias 0 -> 3
- net RTS: track 1.98 -> 26.9 mm, vias 0 -> 1
- net GND: track 134.1 -> 142.5 mm, vias 130 -> 154
- net +3V3: track 31.0 -> 25.9 mm, vias 20 -> 23
- net D-: track 24.3 -> 28.9 mm, vias 1 -> 2
- net D+: track 23.7 -> 27.7 mm, vias 1 -> 2
- net +5V: track 24.5 -> 21.4 mm
- net GSM_RX: track 7.92 -> 9.61 mm
- net NETSTAT_5V: track 14.8 -> 16.5 mm
- net IO0: track 72.3 -> 70.9 mm
- net N$6: track 8.76 -> 7.56 mm
- net N$13: track 5.62 -> 4.52 mm
- net RI_5V: track 30.6 -> 31.7 mm
- net ESP_EN: track 6.50 -> 5.57 mm
- net PWRSTAT_5V: track 35.4 -> 36.2 mm
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- added copper zone on layer 1, net N$1
- added copper zone on layer 1, net V_IN
- added copper zone on layer 16, net V_IN
- removed copper zone on layer 1, net VBUS
- removed copper zone on layer 16, net VBUS
Other:
- outline, holes or cut-outs redrawn
- board text added: "/Users/mcleans/Desktop/Logo-Files-01.bmp"

Commit message: Added CAM files
Routing:
- net GND: track 142.5 -> 139.8 mm
- net +5V: track 21.4 -> 21.9 mm
Changed lines of the file:
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@@
 <drawing>
 <settings>
-<setting alwaysvectorfont="yes"/>
+<setting alwaysvectorfont="no"/>
 <setting verticaltext="up"/>
 </settings>
@@
 <wire x1="32.779365625" y1="22.596228125" x2="33.147" y2="22.206" width="0.8" layer="1"/>
 <via x="33.147" y="22.206" extent="1-16" drill="0.35"/>
-<wire x1="15.763" y1="4.191" x2="15.748" y2="4.206" width="0.4" layer="1"/>
 <wire x1="16.413" y1="4.191" x2="18.088" y2="4.191" width="0.4" layer="1"/>
 <wire x1="18.088" y1="4.191" x2="18.213" y2="4.066" width="0.4" layer="1"/>
-<wire x1="22.262" y1="30.909" x2="24.844" y2="30.909" width="0.6" layer="1"/>
-<wire x1="24.844" y1="30.909" x2="24.892" y2="30.861" width="0.6" layer="1"/>
 <wire x1="27.462" y1="30.909" x2="24.862" y2="30.909" width="0.6" layer="1"/>
 <wire x1="27.462" y1="30.909" x2="29.718" y2="30.909" width="0.6" layer="1"/>
@@
 <wire x1="9.0863125" y1="10.6426" x2="8.6799125" y2="11.049" width="0.4" layer="1"/>
 <via x="8.128" y="11.049" extent="1-16" drill="0.35"/>
-<wire x1="9.5504" y1="10.6426" x2="9.5758" y2="10.668" width="0.4" layer="1"/>
 <via x="14.917" y="21.19" extent="1-16" drill="0.35"/>
 <wire x1="16.09" y1="9.906" x2="17.018" y2="9.906" width="0.4" layer="1"/>
@@
 <contactref element="IC2" pad="4"/>
 <contactref element="CHRG" pad="A"/>
-<wire x1="8.128" y1="27.051" x2="8.509" y2="27.432" width="0.6" layer="1"/>
-<wire x1="8.509" y1="27.432" x2="8.5658" y2="27.4888" width="0.4" layer="1"/>
 <wire x1="8.74" y1="28.9763125" x2="8.5658" y2="28.8021125" width="0.4" layer="1"/>
 <wire x1="8.74" y1="28.9763125" x2="8.74" y2="29.564" width="0.4" layer="1"/>
-<wire x1="8.5658" y1="27.4888" x2="8.5658" y2="28.8021125" width="0.4" layer="1"/>
+<wire x1="8.5658" y1="28.8021125" x2="8.5658" y2="27.4888" width="0.4" layer="1"/>
 <via x="8.74" y="29.564" extent="1-16" drill="0.35"/>
 <wire x1="8.74" y1="29.564" x2="9.4589125" y2="29.564" width="0.4" layer="16"/>
@@
 <via x="11.557" y="14.605" extent="1-16" drill="0.35"/>
 <wire x1="14.3546875" y1="15.621" x2="14.439" y2="15.621" width="0.4" layer="1"/>
-<wire x1="14.439" y1="15.621" x2="14.605" y2="15.787" width="0.4" layer="1"/>
 <polygon width="0.1" layer="16">
 <vertex x="11.938" y="16.383"/>
@@
 <wire x1="15.963" y1="14.097" x2="17.321" y2="12.739" width="0.4" layer="16"/>
 <wire x1="17.321" y1="12.739" x2="17.907" y2="12.739" width="0.4" layer="16"/>
+<wire x1="7.874" y1="26.797" x2="7.493" y2="26.797" width="0.4" layer="1"/>
+<wire x1="8.5658" y1="27.4888" x2="7.874" y2="26.797" width="0.4" layer="1"/>
 </signal>
 <signal name="+3V3" class="1">
