File: src/noise_monitor.sch (EAGLE design)
At the start: 70 parts, among them IC2 MCP73831/OT, T1 S8050, T2 S8050, U2 TEXAS_INSTRUMENTS_SN74HC125TE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, U4 ESP8266-12E/ESP-12E, U5 CP2102N-A02-GQFN28, U6 LP2989AILD-3.3, X2 SIMLOCK-C707_10M006_512_2

Commit message: Fixed DRC
Parts:
- removed MICRO_USB: 10118192-0001LF, noise_tracker:10118192-0001LF
- removed S1, S2: KMR621NGLFS, AQ_sensor_GSM:KMR621NGLFS
- added D7: ON_SEMI_1N4148WSON_SEMI_1N4148WS_0_0, noise_monitor:ON_SEMI_1N4148WSON_SEMI_1N4148WS_0_0
- added FLASH, RESET: KMR621NGLFS, noise_monitor:KMR621NGLFS
- added MICRO-USB: 10118192-0001LF, noise_monitor:10118192-0001LF
- added R23: 0R, rcl:R-EU_R0201
- CN1: device AQ_sensor_GSM:JST_2PIN-SMT-RA -> noise_monitor:JST_2PIN-SMT-RA
- D1, D4: device noise_tracker:ON_SEMI_1N4148WSON_SEMI_1N4148WS_0_0 -> noise_monitor:ON_SEMI_1N4148WSON_SEMI_1N4148WS_0_0
- D2: device noise_tracker:ON_SEMICONDUCTOR_MMSZ5231BT1GON_SEMICONDUCTOR_MMSZ5231BT1G_0_0 -> noise_monitor:ON_SEMICONDUCTOR_MMSZ5231BT1GON_SEMICONDUCTOR_MMSZ5231BT1G_0_0
- D3: device noise_tracker:SEMTECH_SMF05CSEMTECH_SMF05C_0_0 -> noise_monitor:SEMTECH_SMF05CSEMTECH_SMF05C_0_0
- D5, D6: device AQ_sensor_GSM:ON_SEMI_1N4148WSON_SEMI_1N4148WS_0_0 -> noise_monitor:ON_SEMI_1N4148WSON_SEMI_1N4148WS_0_0
- IC2: device noise_tracker:MCP73831/OT -> noise_monitor:MCP73831/OT
- MK2: device noise_tracker:SPH0645LM4H-B -> noise_monitor:SPH0645LM4H-B
- POWER: device AQ_sensor_GSM:PCM12SMTR -> noise_monitor:PCM12SMTR
- T1, T2: device noise_tracker:MMUN2214LT1-NPN-SC59-BEC -> noise_monitor:MMUN2214LT1-NPN-SC59-BEC
- U1: device noise_tracker:GSM_SIM800L -> noise_monitor:GSM_SIM800L
- U2: device noise_tracker:TEXAS_INSTRUMENTS_SN74HC125TEXAS_INSTRUMENTS_SN74HC125_0_0 -> noise_monitor:TEXAS_INSTRUMENTS_SN74HC125TEXAS_INSTRUMENTS_SN74HC125_0_0
- U4: device noise_tracker:ESP8266-12E/ESP-12E -> noise_monitor:ESP8266-12E/ESP-12E
- U5: device CP2102N-A02-GQFN28:CP2102N-A02-GQFN28 -> noise_monitor:CP2102N-A02-GQFN28
- U6: device LP2989AILD-3.3:LP2989AILD-3.3 -> noise_monitor:LP2989AILD-3.3
- X1: device AQ_sensor_GSM:SMACONNECTOR_EDGE_UFL -> noise_monitor:SMACONNECTOR_EDGE_UFL
- X2: device noise_tracker:SIMLOCK-C707_10M006_512_2 -> noise_monitor:SIMLOCK-C707_10M006_512_2
- renumbered CRG to CHRG, TP1 to 5V, TP2 to GND, TP3 to 3V3, TP4 to V-LIPO
Connections:
- removed net VBUS: MICRO_USB.VUSB, POWER.1
- new net N$1: C12.2, C13.2, R23.2, U5.VDD
- new net VB: U1.VBUS
- new net V_IN: D7.CATHODE, MICRO-USB.VUSB, POWER.1
- net +3V3: now also R23.1; no longer C12.2, C13.2, U5.VDD
- net D+: now also MICRO-USB.D+; no longer MICRO_USB.D+
- net D-: now also MICRO-USB.D-; no longer MICRO_USB.D-
- net ESP_RST: now also RESET.1; no longer S2.1
- net GND: now also D7.ANODE, FLASH.2, MICRO-USB.GND, MICRO-USB.ID, MICRO-USB.SHIELD, RESET.2; no longer MICRO_USB.GND, MICRO_USB.ID, MICRO_USB.SHIELD, S1.2, S2.2
- net IO0: now also FLASH.1; no longer S1.1
